Commit message: Change joint_1 to revolute

File: kinova_description/urdf/j2s7s200.xacro (robot description, xacro)
@@ -46,5 +46,5 @@
     <xacro:property name="joint_base_origin_rpy" value="0 0 0" />
     <xacro:property name="joint_1" value="joint_1" />
-    <xacro:property name="joint_1_type" value="continuous" />
+    <xacro:property name="joint_1_type" value="revolute" />
     <xacro:property name="joint_1_axis_xyz" value="0 0 1" />
     <xacro:property name="joint_1_origin_xyz" value="0 0 0.15675" />
