Commit message: kinova_description: corrected type in mimic finger joint

File: kinova_description/urdf/kinova_common.xacro (robot description, xacro)
@@ -81,5 +81,5 @@
             <origin xyz="0.044 -0.003 0" rpy="0 0 0"/>
             <limit lower="0" upper="2" effort="30" velocity="5"/>
-            <mimic joint="${J_PI/180*40}" multiplier="1.0" offset="0.0"/>
+            <mimic joint="${prefix}_joint_finger_${finger_number}" multiplier="${J_PI/180*40}"  offset="0.0"/>
         </joint>
     </xacro:macro>

Commit message: kinova_description: corrected typo in mimic finger joint

File: kinova_description/urdf/kinova_common.xacro (robot description, xacro)
@@ -81,5 +81,5 @@
             <origin xyz="0.044 -0.003 0" rpy="0 0 0"/>
             <limit lower="0" upper="2" effort="30" velocity="5"/>
-            <mimic joint="${prefix}_joint_finger_${finger_number}" multiplier="${J_PI/180*40}"  offset="0.0"/>
+            <!-- mimic joint="${prefix}_joint_finger_${finger_number}" multiplier="${J_PI/180*40}"  offset="0.0"/-->
         </joint>
     </xacro:macro>

Commit message: description: added transmissions to simulate with gazebo and ros_control

File: kinova_description/urdf/kinova_common.xacro (robot description, xacro)
@@ -14,4 +14,9 @@
 	xmlns:xacro="http://ros.org/wiki/xacro">
     <xacro:property name="J_PI" value="3.1415926535897931" />
+	<xacro:macro name="cylinder_inertia" params="m r h">
+		<inertia	ixx="${m*(3*r*r+h*h)/12}" ixy="0" ixz="0"
+					iyy="${m*(3*r*r+h*h)/12}" iyz="0"
+					izz="${m*r*r/2}" />
+	</xacro:macro>
     <xacro:macro name="kinova_armlink" params="link_name link_mesh">
         <link name="${link_name}">
@@ -31,4 +36,9 @@
                 </geometry>
             </collision>
+      <inertial>
+        <mass value="0.01" />
+        <origin xyz="0 0 0" />
+        <cylinder_inertia  m="0.01" r="0.01" h="0.01" />
+      </inertial>
         </link>
     </xacro:macro>
@@ -41,4 +51,19 @@
         <origin xyz="${joint_origin_xyz}" rpy="${joint_origin_rpy}"/>
      </joint>
+     </xacro:macro>
+     <xacro:macro name="kinova_armtransmission" params="joint_name">
+     <transmission name="${joint_name}_trans">
+			<type>transmission_interface/SimpleTransmission</type>
+			<joint name="${joint_name}">
+				<!-- for the gazebo plugin -->
+				<!--hardwareInterface>EffortJointInterface</hardwareInterface-->
+				<!-- for ros control controller -->
+				<hardwareInterface>PositionJointInterface</hardwareInterface>
+			</joint>
+			<actuator name="${joint_name}_motor">
+				<mechanicalReduction>1</mechanicalReduction>
+				<motorTorqueConstant>1</motorTorqueConstant>
+			</actuator>
+		</transmission>
     </xacro:macro>
     <xacro:macro name="kinova_virtual_link" params="link_name">
@@ -46,10 +71,10 @@
             <visual>
                 <geometry>
-                    <box size = "0 0 0"/>
+                    <box size="0.01 0.01 0.01"/>
                 </geometry>
             </visual>
             <collision>
                 <geometry>
-                    <box size = "0 0 0"/>
+                    <box size="0.01 0.01 0.01"/>
                 </geometry>
             </collision>
@@ -74,4 +99,17 @@
             <limit lower="0" upper="2" effort="30" velocity="5"/>
         </joint>
+     <transmission name="${prefix}_joint_finger_${finger_number}_trans">
+			<type>transmission_interface/SimpleTransmission</type>
+			<joint name="${prefix}_joint_finger_${finger_number}">
+				<!-- for the gazebo plugin -->
+				<!--hardwareInterface>EffortJointInterface</hardwareInterface-->
+				<!-- for ros control controller -->
+				<hardwareInterface>PositionJointInterface</hardwareInterface>
+			</joint>
+			<actuator name="${prefix}_joint_finger_${finger_number}_motor">
+				<mechanicalReduction>1</mechanicalReduction>
+				<motorTorqueConstant>1</motorTorqueConstant>
+			</actuator>
+		</transmission>
         <xacro:kinova_armlink link_name="${prefix}_link_finger_tip_${finger_number}" link_mesh="finger_distal"/>
         <joint name="${prefix}_joint_finger_tip_${finger_number}" type="fixed">

File: kinova_description/urdf/m1n6s300.xacro (robot description, xacro)
@@ -89,17 +89,23 @@
         <xacro:kinova_armlink link_name="${link_1}" link_mesh="${link_1_mesh}"/>
         <xacro:kinova_armjoint joint_name="${joint_1}" type="${joint_1_type}" parent="${link_base}" child="${link_1}" joint_axis_xyz="${joint_1_axis_xyz}" joint_origin_xyz="${joint_1_origin_xyz}" joint_origin_rpy="${joint_1_origin_rpy}" joint_lower_limit="${joint_1_lower_limit}" joint_upper_limit="${joint_1_upper_limit}"/>
+        <xacro:kinova_armtransmission joint_name="${joint_1}" />
         <xacro:kinova_armlink link_name="${link_2}" link_mesh="${link_2_mesh}"/>
         <xacro:kinova_armjoint joint_name="${joint_2}" type="${joint_2_type}" parent="${link_1}" child="${link_2}" joint_axis_xyz="${joint_2_axis_xyz}" joint_origin_xyz="${joint_2_origin_xyz}" joint_origin_rpy="${joint_2_origin_rpy}" joint_lower_limit="${joint_2_lower_limit}" joint_upper_limit="${joint_2_upper_limit}"/>
+        <xacro:kinova_armtransmission joint_name="${joint_2}" />
         <xacro:kinova_armlink link_name="${link_3}" link_mesh="${link_3_mesh}"/>
         <xacro:kinova_armjoint joint_name="${joint_3}" type="${joint_3_type}" parent="${link_2}" child="${link_3}" joint_axis_xyz="${joint_3_axis_xyz}" joint_origin_xyz="${joint_3_origin_xyz}" joint_origin_rpy="${joint_3_origin_rpy}" joint_lower_limit="${joint_3_lower_limit}" joint_upper_limit="${joint_3_upper_limit}"/>
+        <xacro:kinova_armtransmission joint_name="${joint_3}" />
         <xacro:kinova_armlink link_name="${link_4}" link_mesh="${link_4_mesh}"/>
         <xacro:kinova_armjoint joint_name="${joint_4}" type="${joint_4_type}" parent="${link_3}" child="${link_4}" joint_axis_xyz="${joint_4_axis_xyz}" joint_origin_xyz="${joint_4_origin_xyz}" joint_origin_rpy="${joint_4_origin_rpy}" joint_lower_limit="${joint_4_lower_limit}" joint_upper_limit="${joint_4_upper_limit}"/>
+        <xacro:kinova_armtransmission joint_name="${joint_4}" />
         <xacro:kinova_armlink link_name="${link_5}" link_mesh="${link_5_mesh}"/>
         <xacro:kinova_armjoint joint_name="${joint_5}" type="${joint_5_type}" parent="${link_4}" child="${link_5}" joint_axis_xyz="${joint_5_axis_xyz}" joint_origin_xyz="${joint_5_origin_xyz}" joint_origin_rpy="${joint_5_origin_rpy}" joint_lower_limit="${joint_5_lower_limit}" joint_upper_limit="${joint_5_upper_limit}"/>
+        <xacro:kinova_armtransmission joint_name="${joint_5}" />
         <xacro:kinova_armlink link_name="${link_6}" link_mesh="${link_6_mesh}"/>
         <xacro:kinova_armjoint joint_name="${joint_6}" type="${joint_6_type}" parent="${link_5}" child="${link_6}" joint_axis_xyz="${joint_6_axis_xyz}" joint_origin_xyz="${joint_6_origin_xyz}" joint_origin_rpy="${joint_6_origin_rpy}" joint_lower_limit="${joint_6_lower_limit}" joint_upper_limit="${joint_6_upper_limit}"/>
+        <xacro:kinova_armtransmission joint_name="${joint_6}" />
         <xacro:kinova_virtual_link link_name="${link_end_effector}"/>
         <xacro:kinova_virtual_joint joint_name="${joint_end_effector}" type="${joint_end_effector_type}" parent="${link_6}" child="${link_end_effector}" joint_axis_xyz="${joint_end_effector_axis_xyz}" joint_origin_xyz="${joint_end_effector_origin_xyz}" joint_origin_rpy="${joint_end_effector_origin_rpy}" joint_lower_limit="0" joint_upper_limit="0"/>
+        <xacro:kinova_3fingers link_hand="${link_6}" prefix="${prefix}"/>
     </xacro:macro>
-    <xacro:kinova_3fingers link_hand="${link_6}" prefix="${prefix}"/>
 </root>

Commit message: kinova_description: fixed kinova_common urdf kinova joint description

File: kinova_description/urdf/kinova_common.xacro (robot description, xacro)
@@ -44,10 +44,44 @@
       </link>
     </xacro:macro>
-  <xacro:macro name="kinova_armjoint" params="joint_name type parent child joint_axis_xyz joint_origin_xyz joint_origin_rpy joint_lower_limit joint_upper_limit joint_velocity_limit joint_torque_limit fixed:=false">
+    <!--
+    We use dummy default values for values only required when type=='revolute':
+    joint_lower_limit and joint_upper_limit (set to 1234567890)
+    We check during macro execution that these values have been set properly if
+    the joint type requires it (revolute).
+    Similarly, we check that velocity and torque limits are set unless the joint
+    type is fixed, and that the fixed parameter is set consistently.
+  -->
+  <xacro:property name="dummy_default_value" value="1234567890"/>
+  <xacro:macro name="kinova_armjoint" params="joint_name
+                                              type
+                                              parent
+                                              child
+                                              joint_axis_xyz
+                                              joint_origin_xyz
+                                              joint_origin_rpy
+                                              joint_lower_limit:=${dummy_default_value}
+                                              joint_upper_limit:=${dummy_default_value}
+                                              joint_velocity_limit:=${dummy_default_value}
+                                              joint_torque_limit:=${dummy_default_value}
+                                              fixed:=false">
+    <xacro:if value="${(type == 'fixed' and not fixed) or (type != 'fixed' and fixed)}"><xacro:ERROR_inconsistent_joint_type_specification/></xacro:if>
+    <xacro:if value="${type == 'revolute'}">
+      <xacro:if value="${joint_lower_limit == dummy_default_value}"><xacro:ERROR_joint_lower_limit_needs_to_be_set_for_a_revolute_joint/></xacro:if>
+      <xacro:if value="${joint_upper_limit == dummy_default_value}"><xacro:ERROR_joint_upper_limit_needs_to_be_set_for_a_revolute_joint/></xacro:if>
+    </xacro:if>
+    <xacro:unless value="${type =='fixed'}">
+      <xacro:if value="${joint_velocity_limit == dummy_default_value}"><xacro:ERROR_joint_velocity_limit_needs_to_be_set_for_a_non_fixed_joint/></xacro:if>
+      <xacro:if value="${joint_torque_limit == dummy_default_value}"><xacro:ERROR_joint_torque_limit_needs_to_be_set_for_a_non_fixed_joint/></xacro:if>
+    </xacro:unless>
     <joint name="${joint_name}" type="${type}">
         <parent link="${parent}"/>
         <child link="${child}"/>
         <axis xyz="${joint_axis_xyz}"/>
+        <xacro:if value="${type == 'revolute'}">
         <limit effort="${joint_torque_limit}" velocity="${joint_velocity_limit}" lower="${joint_lower_limit}" upper="${joint_upper_limit}"/>
+        </xacro:if>
+        <xacro:if value="${type == 'continuous'}">
+        <limit effort="${joint_torque_limit}" velocity="${joint_velocity_limit}"/>
+        </xacro:if>
         <origin xyz="${joint_origin_xyz}" rpy="${joint_origin_rpy}"/>
         <dynamics damping="0.0" friction="0.0"/>
@@ -85,5 +119,7 @@
         <child link="${child}"/>
         <axis xyz="${joint_axis_xyz}"/>
+        <xacro:unless value="${type == 'fixed'}">
         <limit effort="2000" velocity="1" lower="${joint_lower_limit}" upper="${joint_upper_limit}"/>
+        </xacro:unless>
         <origin xyz="${joint_origin_xyz}" rpy="${joint_origin_rpy}"/>
      </joint>
